File: luther.sch (KiCad schematic (older format))
At the start: 6 parts, among them J1 Conn_01x02, U1 Teensy4.0, U2 RFM95W_LoRa_Radio, U3 VHN5019_Breakout, U4 VHN5019_Breakout, U5 bno055

Commit message: misc changes
Parts:
- removed U5: bno055, NUSTARS Libs:bno055, symbol NUSTARS:bno055
- added D1: LED, symbol Device:LED
- added J2: SMART_AUDIO, symbol Connector_Generic:Conn_01x02
- added J3: SERVO_LEVER, Connector_JST:JST_PH_B3B-PH-K_1x03_P2.00mm_Vertical, symbol Connector_Generic:Conn_01x03
- added J4: SERVO_CLOCK, Connector_JST:JST_PH_B3B-PH-K_1x03_P2.00mm_Vertical, symbol Connector_Generic:Conn_01x03
- added R1: 330, symbol Device:R_Small_US
- added SW1: SW_SPST, NUSTARS Libs:GF-123-0054, symbol Switch:SW_SPST
- added U5: VHN5019_Breakout, NUSTARS Libs:VNH5019_breakout, symbol NUSTARS:VHN5019_Breakout
- added U6, U7: BUCK, symbol NUSTARS:BUCK
Connections:
- net labels added: 3V3B, M0_INA, M0_INB, M0_PWM, M1_INA, M1_INB, M1_PWM, M2_INA, M2_INB, M2_PWM
- net labels removed: FNA2T, T2FNA
- wire segments 5 -> 26
Other:
- note removed: "Consider hooking this up to 3.3V buck output\n"
- moved on the sheet: J1, U2, U3, U4

Commit message: updates
Parts:
- removed J2: SMART_AUDIO, symbol Connector_Generic:Conn_01x02
- removed U3, U4, U5: VHN5019_Breakout, NUSTARS Libs:VNH5019_breakout, symbol NUSTARS:VHN5019_Breakout
- removed U7: BUCK, symbol NUSTARS:BUCK
- added H1, H2, H3, H4: MountingHole, MountingHole:MountingHole_3.2mm_M3, symbol Mechanical:MountingHole
- added J2: SERVO_WIRE, Connector_JST:JST_PH_B3B-PH-K_1x03_P2.00mm_Vertical, symbol Connector_Generic:Conn_01x03
- added J5: DRV_MOTOR0, Connector_JST:JST_PH_B2B-PH-K_1x02_P2.00mm_Vertical, symbol Connector_Generic:Conn_01x02
- added J6: DRV_MOTOR1, Connector_JST:JST_PH_B2B-PH-K_1x02_P2.00mm_Vertical, symbol Connector_Generic:Conn_01x02
- added J7: Antenna, NUSTARS Libs:Antenna, symbol Connector:Conn_01x01_Male
- added Q1, Q2: GSD, Package_TO_SOT_SMD:SOT-23_Handsoldering, symbol Device:Q_NMOS_GSD
- added U3, U5: drv8838_breakout, NUSTARS Libs:drv8838_breakout, symbol DRV:drv8838_breakout
- D1: footprint (none) -> LED_SMD:LED_1206_3216Metric_Pad1.42x1.75mm_HandSolder
- R1: footprint (none) -> Resistor_SMD:R_1206_3216Metric_Pad1.42x1.75mm_HandSolder
- U6: footprint (none) -> NUSTARS Libs:D24V50F5
Connections:
- net 3V3B is gone; now on net 3V3T: U2.1 (Vin)
- net 3V3T: now also U3.2 (VCC), U5.2 (VCC)
- net GND: now also Q1.2 (S), Q2.2 (S), U3.1 (GND), U3.10 (GND), U5.1 (GND), U5.10 (GND); no longer J3.2 (Pin_2)
- net M0_PWM: now also U3.3 (ENABLE)
- net M1_PWM: now also U5.3 (ENABLE)
- net VBAT: now also J2.1 (Pin_1), U3.9 (VIN), U5.9 (VIN)
- net SRV_L_PWM: now reaches J3.3 (Pin_3)
- net SRV_L_PWM: no longer U1.~ (GND)
- net SRV_C_PWM: now reaches J4.3 (Pin_3)
- net SRV_C_PWM: no longer U1.~ (GND)
- net LORA_ANTENNA: now reaches U2.15 (Antenna)
- net LORA_ANTENNA: now also J7.1 (Pin_1)
- new net: J6.1 (Pin_1), U5.7 (OUT1)
- new net: J6.2 (Pin_2), U5.8 (OUT2)
- new net: J5.1 (Pin_1), U3.7 (OUT1)
- new net: J5.2 (Pin_2), U3.8 (OUT2)
- new net: J3.2 (Pin_2), Q1.3 (D)
- new net: J2.2 (Pin_2), Q2.3 (D)
- new net M0_DIR: U3.4 (PHASE)
- new net M0_DISABLE: U3.5 (NOT_SLEEP)
- new net M1_DIR: U5.4 (PHASE)
- new net M1_DISABLE: U5.5 (NOT_SLEEP)
- new net SRV_W_PWM: J2.3 (Pin_3)
- new net S_L_NMOS: Q1.1 (G)
- new net S_W_NMOS: Q2.1 (G)
- now unconnected: U1.~ (GND)
Other:
- moved on the sheet: D1, J1, J3, J4, R1, SW1, U1, U2, U6

Commit message: prelim finish sans decor
Parts:
- removed H4: MountingHole, MountingHole:MountingHole_3.2mm_M3, symbol Mechanical:MountingHole
- added J2: Conn_01x04, Connector_JST:JST_PH_B4B-PH-K_1x04_P2.00mm_Vertical, symbol Connector_Generic:Conn_01x04
- J1: value Conn_01x02 -> BAT
- renumbered J4 to CLOCK1, J3 to LEVER1, J2 to WIRE1
Connections:
- net SRV_C_PWM is gone; now on net S_C_PWM: CLOCK1.3 (Pin_3)
- net SRV_L_PWM is gone; now on net S_L_PWM: LEVER1.3 (Pin_3)
- net SRV_W_PWM is gone; now on net S_W_PWM: WIRE1.3 (Pin_3)
- net 3V3T: now also J2.1 (Pin_1)
- net GND: now also J2.2 (Pin_2)
- net M0_DIR: now also U1.8 (6_OUT1D)
- net M0_DISABLE: now also U1.9 (7_RX2_OUT1A)
- net M0_PWM: now also U1.7 (5_IN2)
- net M1_DIR: now also U1.5 (3_LRCLK2)
- net M1_DISABLE: now also U1.6 (4_BCLK2)
- net M1_PWM: now also U1.4 (2_OUT2)
- net SCL: now also J2.3 (Pin_3)
- net SDA: now also J2.4 (Pin_4)
- net S_L_NMOS: now also U1.28 (21_A7_RX5_BCLK1)
- net S_W_NMOS: now also U1.30 (23_A9_CRX1_MCLK1)
- net S_C_PWM: now reaches U1.21 (14_A0_TX3_SPDIF_OUT)
- net S_L_PWM: now reaches U1.22 (15_A1_RX3_SPDIF_IN)
- net S_W_PWM: now reaches U1.29 (22_A8_CTX1)
Changed lines of the file:
@@
 EESchema Schematic File Version 4
+LIBS:luther-cache
 EELAYER 30 0
 EELAYER END
@@
 P 8800 1150
 F 0 "J1" H 8880 1142 50  0000 L CNN
-F 1 "Conn_01x02" H 8880 1051 50  0000 L CNN
+F 1 "BAT" H 8880 1051 50  0000 L CNN
 F 2 "NUSTARS Libs:DEANS" H 8800 1150 50  0001 C CNN
 F 3 "~" H 8800 1150 50  0001 C CNN
@@
 GND
 $Comp
-L Connector_Generic:Conn_01x03 J3
+L Connector_Generic:Conn_01x03 LEVER1
 U 1 1 5E2412EE
 P 7300 5700
-F 0 "J3" H 7380 5742 50  0000 L CNN
+F 0 "LEVER1" H 7380 5742 50  0000 L CNN
 F 1 "SERVO_LEVER" H 7380 5651 50  0000 L CNN
 F 2 "Connector_JST:JST_PH_B3B-PH-K_1x03_P2.00mm_Vertical" H 7300 5700 50  0001 C CNN
@@
 M0_DISABLE
 $Comp
-L Connector_Generic:Conn_01x03 J2
+L Connector_Generic:Conn_01x03 WIRE1
 U 1 1 5E24D9D0
 P 7300 5300
-F 0 "J2" H 7380 5342 50  0000 L CNN
+F 0 "WIRE1" H 7380 5342 50  0000 L CNN
 F 1 "SERVO_WIRE" H 7380 5251 50  0000 L CNN
 F 2 "Connector_JST:JST_PH_B3B-PH-K_1x03_P2.00mm_Vertical" H 7300 5300 50  0001 C CNN
@@
 GND
 $Comp
-L Connector_Generic:Conn_01x03 J4
+L Connector_Generic:Conn_01x03 CLOCK1
 U 1 1 5E241714
 P 7300 6100
-F 0 "J4" H 7380 6142 50  0000 L CNN
+F 0 "CLOCK1" H 7380 6142 50  0000 L CNN
 F 1 "SERVO_CLOCK" H 7380 6051 50  0000 L CNN
 F 2 "Connector_JST:JST_PH_B3B-PH-K_1x03_P2.00mm_Vertical" H 7300 6100 50  0001 C CNN
@@
 $EndComp
 Text GLabel 7100 5400 0    50   Input ~ 0
-SRV_W_PWM
+S_W_PWM
 Text GLabel 7100 5800 0    50   Input ~ 0
-SRV_L_PWM
+S_L_PWM
 Text GLabel 7100 6200 0    50   Input ~ 0
-SRV_C_PWM
+S_C_PWM
 Wire Wire Line
 	6000 5700 7100 5700
@@
 	1    0    0    -1
 $EndComp
-$Comp
-L Mechanical:MountingHole H4
-U 1 1 5E2DD8C1
-P 10300 1500
-F 0 "H4" H 10400 1546 50  0000 L CNN
-F 1 "MountingHole" H 10400 1455 50  0000 L CNN
-F 2 "MountingHole:MountingHole_3.2mm_M3" H 10300 1500 50  0001 C CNN
-F 3 "~" H 10300 1500 50  0001 C CNN
-	1    10300 1500
-	1    0    0    -1
-$EndComp
 Text GLabel 8450 4300 2    50   Input ~ 0
 LORA_ANTENNA
@@
 Wire Wire Line
 	8200 4300 8450 4300
+Text GLabel 2450 1450 0    50   Input ~ 0
+M1_PWM
+Text GLabel 2450 1550 0    50   Input ~ 0
+M1_DIR
+Text GLabel 2450 1650 0    50   Input ~ 0
+M1_DISABLE
+Text GLabel 2450 1750 0    50   Input ~ 0
+M0_PWM
+Text GLabel 2450 1850 0    50   Input ~ 0
+M0_DIR
+Text GLabel 2450 1950 0    50   Input ~ 0
+M0_DISABLE
+$Comp
+L Connector_Generic:Conn_01x04 J2
+U 1 1 5E23D450
+P 5700 2450
+F 0 "J2" H 5780 2442 50  0000 L CNN
+F 1 "Conn_01x04" H 5780 2351 50  0000 L CNN
+F 2 "Connector_JST:JST_PH_B4B-PH-K_1x04_P2.00mm_Vertical" H 5700 2450 50  0001 C CNN
+F 3 "~" H 5700 2450 50  0001 C CNN
+	1    5700 2450
+	1    0    0    -1
+$EndComp
+Text GLabel 5500 2350 0    50   Input ~ 0
+3V3T
+Text GLabel 5500 2450 0    50   Input ~ 0
+GND
+Text GLabel 5500 2550 0    50   Input ~ 0
+SCL
+Text GLabel 5500 2650 0    50   Input ~ 0
+SDA
+Text GLabel 4650 3750 2    50   Input ~ 0
+S_W_NMOS
+Text GLabel 4650 3850 2    50   Input ~ 0
+S_W_PWM
+Text GLabel 2450 3850 0    50   Input ~ 0
+S_L_NMOS
+Text GLabel 2450 3250 0    50   Input ~ 0
+S_L_PWM
+Text GLabel 2450 3150 0    50   Input ~ 0
+S_C_PWM
 $EndSCHEMATC
