File: luther.kicad_pcb (KiCad board)
At the start: 2 copper layers, 114 x 50 mm, 6 parts, among them J1 Conn_01x02, U1 Teensy4.0, U2 RFM95W_LoRa_Radio, U3 VHN5019_Breakout, U4 VHN5019_Breakout, U5 bno055

Commit message: misc changes
Parts:
- added J3: SERVO_LEVER, Connector_JST:JST_PH_B3B-PH-K_1x03_P2.00mm_Vertical, F.Cu at (43.0, 148.0)
- added J4: SERVO_CLOCK, Connector_JST:JST_PH_B3B-PH-K_1x03_P2.00mm_Vertical, F.Cu at (60.8, 136.5)
- added SW1: SW_SPST, NUSTARS Libs:GF-123-0054, F.Cu at (40.8, 134.6)
- U5: value bno055 -> VHN5019_Breakout; footprint NUSTARS Libs:bno055 -> NUSTARS Libs:VNH5019_breakout
- moved U5 51.2 mm to (11.5, 134.6), turned to 0 degrees
Connections:
- net Net-(U3-Pad1) renamed M0_INA
- net Net-(U3-Pad3) renamed M0_PWM
- net Net-(U3-Pad6) renamed M0_INB
- net Net-(U4-Pad1) renamed M1_INA
- net Net-(U4-Pad3) renamed M1_PWM
- net Net-(U4-Pad6) renamed M1_INB
- net Net-(U5-Pad3) renamed M2_PWM
- net Net-(U5-Pad6) renamed M2_INB
- J1 pad 1: VBAT -> Net-(J1-Pad1)
- U1 pad 2: FNA2T -> LORA_INT
- U1 pad 3: T2FNA -> LORA_RST
- U2 pad 1: 3V3T -> 3V3B
- U3 pad 13: Net-(U3-Pad13) -> GND
- U3 pad 14: Net-(U3-Pad14) -> VBAT
- U3 pad 7: Net-(U3-Pad7) -> 3V3T
- U3 pad 8: Net-(U3-Pad8) -> GND
- U4 pad 13: Net-(U4-Pad13) -> GND
- U4 pad 14: Net-(U4-Pad14) -> VBAT
- U4 pad 7: Net-(U4-Pad7) -> 3V3T
- U4 pad 8: Net-(U4-Pad8) -> GND
- U5 pad 1: 3V3T -> M2_INA
- U5 pad 4: SDA -> Net-(U5-Pad4)
- U5 pad 5: SCL -> Net-(U5-Pad5)
- U5 pad 7: Net-(U5-Pad7) -> 3V3T
- U5 pad 8: Net-(U5-Pad8) -> GND

Commit message: updates
Parts:
- removed U4: VHN5019_Breakout, NUSTARS Libs:VNH5019_breakout
- added D1: LED, LED_SMD:LED_1206_3216Metric_Pad1.42x1.75mm_HandSolder, F.Cu at (65.0, 105.0)
- added H1: MountingHole, MountingHole:MountingHole_3.2mm_M3, F.Cu at (34.0, 74.0)
- added H2: MountingHole, MountingHole:MountingHole_3.2mm_M3, F.Cu at (34.0, 116.0)
- added H3: MountingHole, MountingHole:MountingHole_3.2mm_M3, F.Cu at (97.0, 116.0)
- added H4: MountingHole, MountingHole:MountingHole_3.2mm_M3, F.Cu at (136.0, 71.0)
- added J2: SERVO_WIRE, Connector_JST:JST_PH_B3B-PH-K_1x03_P2.00mm_Vertical, F.Cu at (78.0, 75.0)
- added J5: DRV_MOTOR0, Connector_JST:JST_PH_B2B-PH-K_1x02_P2.00mm_Vertical, F.Cu at (46.0, 75.0)
- added J6: DRV_MOTOR1, Connector_JST:JST_PH_B2B-PH-K_1x02_P2.00mm_Vertical, F.Cu at (56.0, 75.0)
- added J7: Antenna, NUSTARS Libs:Antenna, F.Cu at (109.0, 96.0)
- added Q1: GSD, Package_TO_SOT_SMD:SOT-23_Handsoldering, F.Cu at (91.0, 82.5)
- added Q2: GSD, Package_TO_SOT_SMD:SOT-23_Handsoldering, F.Cu at (80.0, 82.5)
- added R1: 330, Resistor_SMD:R_1206_3216Metric_Pad1.42x1.75mm_HandSolder, B.Cu at (65.0, 105.0)
- added U6: BUCK, NUSTARS Libs:D24V50F5, F.Cu at (92.0, 100.0)
- U3: value VHN5019_Breakout -> drv8838_breakout; footprint NUSTARS Libs:VNH5019_breakout -> NUSTARS Libs:drv8838_breakout
- U5: value VHN5019_Breakout -> drv8838_breakout; footprint NUSTARS Libs:VNH5019_breakout -> NUSTARS Libs:drv8838_breakout; moved to B.Cu
- moved J3 86.3 mm to (89.0, 75.0)
- moved U5 70.0 mm to (60.0, 84.0), turned to 90 degrees
- moved J4 61.9 mm to (67.0, 75.0)
- moved U3 45.9 mm to (45.0, 84.0), turned to 90 degrees
- moved J1 36.4 mm to (44.0, 109.5), turned to 180 degrees
- moved SW1 33.8 mm to (70.2, 118.0), turned to 180 degrees
- moved U2 25.6 mm to (100.0, 103.0)
- moved U1 3.61 mm to (52.0, 91.0), turned to 180 degrees
Connections:
- net M0_INB renamed Net-(U3-Pad6)
- net M2_INB renamed Net-(U5-Pad6)
- net Net-(J3-Pad3) renamed SRV_L_PWM
- net Net-(J4-Pad3) renamed SRV_C_PWM
- net Net-(U3-Pad4) renamed M0_DIR
- net Net-(U3-Pad5) renamed M0_DISABLE
- net Net-(U5-Pad4) renamed M1_DIR
- net Net-(U5-Pad5) renamed M1_DISABLE
- J3 pad 2: GND -> Net-(J3-Pad2)
- U2 pad 1: 3V3B -> 3V3T
- U2 pad 15: Net-(U2-Pad15) -> LORA_ANTENNA
- U3 pad 1: M0_INA -> GND
- U3 pad 10: Net-(U3-Pad10) -> GND
- U3 pad 2: Net-(U3-Pad2) -> 3V3T
- U3 pad 7: 3V3T -> Net-(J5-Pad1)
- U3 pad 8: GND -> Net-(J5-Pad2)
- U3 pad 9: Net-(U3-Pad9) -> VBAT
- U5 pad 1: M2_INA -> GND
- U5 pad 10: Net-(U5-Pad10) -> GND
- U5 pad 2: Net-(U5-Pad2) -> 3V3T
- U5 pad 3: M2_PWM -> M1_PWM
- U5 pad 7: 3V3T -> Net-(J6-Pad1)
- U5 pad 8: GND -> Net-(J6-Pad2)
- U5 pad 9: Net-(U5-Pad9) -> VBAT
Routing:
- net 5V: track 0.00 -> 61.4 mm
- net 3V3T: track 0.00 -> 42.2 mm
- net SCK: track 0.00 -> 41.3 mm
- net MISO: track 0.00 -> 39.7 mm
- net MOSI: track 0.00 -> 36.1 mm
- net CS: track 0.00 -> 34.0 mm
- net LORA_INT: track 0.00 -> 12.5 mm
- net LORA_RST: track 0.00 -> 11.2 mm
- net Net-(J5-Pad1): track 0.00 -> 6.66 mm
- net Net-(J6-Pad2): track 0.00 -> 6.59 mm
- net Net-(J5-Pad2): track 0.00 -> 6.43 mm
- net Net-(J3-Pad2): track 0.00 -> 6.02 mm
- net Net-(J2-Pad2): track 0.00 -> 6.02 mm
- net Net-(J6-Pad1): track 0.00 -> 5.79 mm
- net LORA_ANTENNA: track 0.00 -> 4.16 mm
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- added copper zone on F.Cu, net GND
- added copper zone on F.Cu, net VBAT
Other:
- board size 114 x 50 mm -> 91 x 50 mm
- board text removed: "5G8"
- board text removed: "EMISSION DIRECTION -->"
- board text removed: "HIGH DENSITY REGION"
- board text removed: "LORA XCLUD"

Commit message: prelim finish sans decor
Parts:
- removed H4: MountingHole, MountingHole:MountingHole_3.2mm_M3
- added J2: Conn_01x04, Connector_JST:JST_PH_B4B-PH-K_1x04_P2.00mm_Vertical, F.Cu at (36.0, 110.0)
- J1: value Conn_01x02 -> BAT
- moved J1 3.00 mm to (47.0, 109.5)
- renumbered J4 to CLOCK1, J3 to LEVER1, J2 to WIRE1
Connections:
- CLOCK1 pad 3: SRV_C_PWM -> S_C_PWM
- LEVER1 pad 3: SRV_L_PWM -> S_L_PWM
- U1 pad 21: Net-(U1-Pad21) -> S_C_PWM
- U1 pad 22: Net-(U1-Pad22) -> S_L_PWM
- U1 pad 28: Net-(U1-Pad28) -> S_L_NMOS
- U1 pad 29: Net-(U1-Pad29) -> S_W_PWM
- U1 pad 30: Net-(U1-Pad30) -> S_W_NMOS
- U1 pad 4: Net-(U1-Pad4) -> M1_PWM
- U1 pad 5: Net-(U1-Pad5) -> M1_DIR
- U1 pad 6: Net-(U1-Pad6) -> M1_DISABLE
- U1 pad 7: Net-(U1-Pad7) -> M0_PWM
- U1 pad 8: Net-(U1-Pad8) -> M0_DIR
- U1 pad 9: Net-(U1-Pad9) -> M0_DISABLE
- WIRE1 pad 3: SRV_W_PWM -> S_W_PWM
Routing:
- net S_L_PWM: track 0.00 -> 75.6 mm
- net S_C_PWM: track 0.00 -> 50.5 mm, vias 0 -> 1
- net S_W_PWM: track 0.00 -> 48.4 mm
- net S_L_NMOS: track 0.00 -> 46.5 mm
- net S_W_NMOS: track 0.00 -> 35.3 mm
- net 3V3T: track 42.2 -> 74.4 mm
- net GND: track 0.00 -> 25.2 mm, vias 9 -> 14
- net SCL: track 0.00 -> 17.8 mm
- net Net-(J1-Pad1): track 0.16 -> 15.0 mm
- net SDA: track 0.00 -> 14.4 mm
- net M0_PWM: track 0.00 -> 10.1 mm
- net M0_DISABLE: track 0.00 -> 10.1 mm
- net M0_DIR: track 0.00 -> 10.1 mm
- net M1_PWM: track 0.00 -> 4.80 mm
- net M1_DISABLE: track 0.00 -> 4.80 mm
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- removed copper zone on F.Cu, net GND
Other:
- board text added: "NUSTARS NSL ROVER CONTROLLER REV 2020-01-18"
